Commit message: update cartpole urdf

File: models/g1_description/g1_7dof_cartpole.urdf (robot description, URDF)
Before this commit: robot g1_29dof, 27 links, 26 joints
Links:
- link cartpole_cart: mass 10 -> 1
- link cartpole_pole: mass 1 -> 0.5
Joints:
- joint cartpole_x: origin xyz=0 0 0 rpy=0 0 0 -> xyz=0.055 0 0 rpy=0 0 0; type prismatic -> fixed
