Commit message: update cartpole

File: koopman/cartpole/models/g1_description/g1_7dof_rubber_hand.urdf (robot description, URDF)
Before this commit: robot g1_29dof, 27 links, 26 joints
Links:
- removed link right_rubber_hand
- added link cart, mass 0.5; visual box size=0.1 0.05 0.05
- added link pole, mass 0.3; visual cylinder length=0.3 radius=0.01
Joints:
- added joint pole_joint: type continuous, parent cart, child pole, origin xyz=0 0 0.05, axis 0 1 0
- joint right_hand_palm_joint: child right_rubber_hand -> cart
