Commit message: update urdf

File: koopman/cartpole/models/g1_description/g1_7dof_cartpole.urdf (robot description, URDF)
Before this commit: robot g1_29dof, 27 links, 26 joints
Links:
- link left_elbow_link: geometry visual mesh filename=meshes/left_elbow_link.obj
- link left_shoulder_pitch_link: geometry visual mesh filename=meshes/left_shoulder_pitch_link.obj
- link left_shoulder_roll_link: geometry visual mesh filename=meshes/left_shoulder_roll_link.obj
- link left_shoulder_yaw_link: geometry visual mesh filename=meshes/left_shoulder_yaw_link.obj
- link left_wrist_pitch_link: geometry visual mesh filename=meshes/left_wrist_pitch_link.obj
- link left_wrist_roll_link: geometry visual mesh filename=meshes/left_wrist_roll_link.obj
- link left_wrist_yaw_link: geometry visual mesh filename=meshes/left_wrist_yaw_link.obj
- link right_elbow_link: geometry visual mesh filename=meshes/right_elbow_link.obj
- link right_shoulder_pitch_link: geometry visual mesh filename=meshes/right_shoulder_pitch_link.obj
- link right_shoulder_roll_link: geometry visual mesh filename=meshes/right_shoulder_roll_link.obj
- link right_shoulder_yaw_link: geometry visual mesh filename=meshes/right_shoulder_yaw_link.obj
- link right_wrist_pitch_link: geometry visual mesh filename=meshes/right_wrist_pitch_link.obj
- link right_wrist_roll_link: geometry visual mesh filename=meshes/right_wrist_roll_link.obj
- link right_wrist_yaw_link: geometry visual mesh filename=meshes/right_wrist_yaw_link.obj

Commit message: add another data collection method

File: koopman/cartpole/models/g1_description/g1_7dof_cartpole.urdf (robot description, URDF)
Before this commit: robot g1_29dof, 27 links, 26 joints
Links:
- link cartpole_cart: mass 0.5 -> 0.1
- link cartpole_pole: mass 0.5 -> 0.1

Commit message: update cartpole

File: koopman/cartpole/models/g1_description/g1_7dof_cartpole.urdf (robot description, URDF)
Before this commit: robot g1_29dof, 28 links, 27 joints
Links:
- removed link cart
- removed link left_rubber_hand
- removed link pole
- added link cartpole_cart, mass 0.1; visual box size=0.03 0.03 0.03
- added link cartpole_pole, mass 0.1; visual cylinder length=0.15 radius=0.005; visual sphere radius=0.015
- link left_elbow_link: geometry visual mesh filename=meshes/left_elbow_link.obj
- link left_shoulder_pitch_link: geometry visual mesh filename=meshes/left_shoulder_pitch_link.obj
- link left_shoulder_roll_link: geometry visual mesh filename=meshes/left_shoulder_roll_link.obj
- link left_shoulder_yaw_link: geometry visual mesh filename=meshes/left_shoulder_yaw_link.obj
- link left_wrist_pitch_link: geometry visual mesh filename=meshes/left_wrist_pitch_link.obj
- link left_wrist_roll_link: geometry visual mesh filename=meshes/left_wrist_roll_link.obj
- link left_wrist_yaw_link: geometry visual mesh filename=meshes/left_wrist_yaw_link.obj
- link right_elbow_link: geometry visual mesh filename=meshes/right_elbow_link.obj
- link right_shoulder_pitch_link: geometry visual mesh filename=meshes/right_shoulder_pitch_link.obj
- link right_shoulder_roll_link: geometry visual mesh filename=meshes/right_shoulder_roll_link.obj
- link right_shoulder_yaw_link: geometry visual mesh filename=meshes/right_shoulder_yaw_link.obj
- link right_wrist_pitch_link: geometry visual mesh filename=meshes/right_wrist_pitch_link.obj
- link right_wrist_roll_link: geometry visual mesh filename=meshes/right_wrist_roll_link.obj
- link right_wrist_yaw_link: geometry visual mesh filename=meshes/right_wrist_yaw_link.obj
Joints:
- removed joint left_hand_palm_joint
- removed joint pole_joint
- removed joint right_hand_palm_joint
- added joint cartpole_theta: type continuous, parent cartpole_cart, child cartpole_pole, origin xyz=0 0 0 rpy=0 0 0, axis 0 -1 0
- added joint cartpole_x: type fixed, parent right_wrist_yaw_link, child cartpole_cart, origin xyz=0.06 0 0 rpy=0 0 0, axis 1 0 0
